Commit message: implement handcrafted policy

File: assets/robots/roller.urdf (robot description, URDF)
Before this commit: robot roller, 12 links, 11 joints
Joints:
- joint joint1_right: limit lower=0.01 upper=0.03 effort=10.0 velocity=10000 -> lower=-0.01 upper=0.03 effort=10.0 velocity=10000
- joint joint4_left: origin xyz=0.0 0.0368 0.0 rpy=0 0 0 -> xyz=0.0 0.0368 0.0 rpy=0 1.57 0
- joint joint4_right: origin xyz=0.0 -0.0368 0.0 rpy=0 0 0 -> xyz=0.0 -0.0368 0.0 rpy=0 1.57 0
- joint joint5_left: origin xyz=0.0 0.0368 0.0 rpy=0 0 0 -> xyz=0.0 0.0368 0.0 rpy=0 1.57 0
- joint joint5_right: origin xyz=0.0 0.0368 0.0 rpy=0 0 0 -> xyz=0.0 0.0368 0.0 rpy=0 1.57 0
- joint wrist: axis 0 0 1 -> 0 0 -1
