Commit message: add gelsight

File: assets/objects/rounded_cube.urdf (robot description, URDF)
Before this commit: robot urdf_robot, 1 links, 0 joints
Links:
- link base_link: mass 0.05 -> 1.0

File: assets/robots/roller.urdf (robot description, URDF)
Before this commit: robot roller, 12 links, 11 joints
Links:
- link link5_left: geometry collision cylinder length=0.05 radius=0.018; visual cylinder length=0.05 radius=0.02
- link link5_right: geometry collision cylinder length=0.05 radius=0.018; visual cylinder length=0.05 radius=0.02
Joints:
- joint joint5_right: origin xyz=0.0 0.0368 0.0 rpy=0 1.57 0 -> xyz=0.0 -0.0368 0.0 rpy=0 1.57 0

File: assets/sensors/roller.urdf (robot description, URDF)
Before this commit: robot digit, 1 links, 0 joints
Links:
- link baseLink: geometry collision cylinder length=0.05 radius=0.02; visual cylinder length=0.05 radius=0.02
